Commit message: Add files via upload

File: description/robot.urdf.xacro (robot description, xacro)
@@ -2,3 +2,4 @@
 <robot xmlns:xacro="http://www.ros.org/wiki/xacro"  name="robot">
    <xacro:include filename="robot_core.xacro" />
+   <xacro:include filename="gazebo_control.xacro" />
 </robot>

File: description/robot_core.xacro (robot description, xacro)
@@ -41,4 +41,7 @@
     </xacro:inertial_box>
  </link>
+ <gazebo reference="chassis">
+    <material>Gazebo/White</material>
+</gazebo>
 <!-- LEFT WHEEL -->
 <joint name="left_wheel_joint" type="continuous">
@@ -64,4 +67,7 @@
     </xacro:inertial_cylinder>
 </link>
+<gazebo reference="left_wheel">
+    <material>Gazebo/Blue</material>
+</gazebo>
 <!-- RIGHT WHEEL -->
 <joint name="right_wheel_joint" type="continuous">
@@ -87,4 +93,7 @@
     </xacro:inertial_sphere>
 </link>
+<gazebo reference="right_wheel">
+    <material>Gazebo/Blue</material>
+</gazebo>
 <!-- CASTER WHEEL -->
 <joint name="caster_wheel_joint" type="fixed">
@@ -106,3 +115,8 @@
     </collision>
 </link>
+<gazebo reference="caster_wheel">
+    <material>Gazebo/White</material>
+    <mu1 value="0.001"/> <!-- 摩擦力設定 -->
+    <mu2 value="0.001"/>
+</gazebo>
 </robot>

Commit message: Add files via upload

File: description/robot.urdf.xacro (robot description, xacro)
@@ -3,3 +3,4 @@
    <xacro:include filename="robot_core.xacro" />
    <xacro:include filename="gazebo_control.xacro" />
+   <xacro:include filename="lidar.xacro" />
 </robot>

File: description/robot_core.xacro (robot description, xacro)
@@ -89,7 +89,7 @@
         </geometry>
     </collision>
-    <xacro:inertial_sphere mass="0.1" radius="0.05">
+     <xacro:inertial_cylinder mass="0.1" length="0.05" radius="0.05">
         <origin xyz="0 0 0" rpy="0 0 0"/>
-    </xacro:inertial_sphere>
+    </xacro:inertial_cylinder>
 </link>
 <gazebo reference="right_wheel">
@@ -114,9 +114,12 @@
         </geometry>
     </collision>
+    <xacro:inertial_sphere mass="0.3" radius="0.05">
+        <origin xyz="0 0 0" rpy="0 0 0"/>
+    </xacro:inertial_sphere>
 </link>
 <gazebo reference="caster_wheel">
     <material>Gazebo/White</material>
-    <mu1 value="0.001"/> <!-- 摩擦力設定 -->
-    <mu2 value="0.001"/>
+    <mu1 value="0.0"/> <!-- 摩擦力設定 -->
+    <mu2 value="0.0"/>
 </gazebo>
 </robot>
