Commit message: Add files via upload

File: description/robot_core.xacro (robot description, xacro)
@@ -49,5 +49,5 @@
     <child link="left_wheel"/>
     <origin xyz="0 0.175 0" rpy="-${pi/2} 0 0"/>
-    <axis xyz="0 0 1"/> ...繞Z逆時針轉+1...
+    <axis xyz="0 0 1"/> ...繞Z逆時針轉...
 </joint>
 <link name="left_wheel">
